Commit message: New release
More realistic simulation environment, including effects of data transfer.

File: models/bittle.urdf (robot description, URDF)
Before this commit: robot Nybble, 9 links, 8 joints
Links:
- added link left_back_paw, mass 0.0005; collision cylinder length=0.01 radius=0.006; visual cylinder length=0.01 radius=0.006
- added link left_front_paw, mass 0.0005; collision cylinder length=0.01 radius=0.006; visual cylinder length=0.01 radius=0.006
- added link right_back_paw, mass 0.0005; collision cylinder length=0.01 radius=0.006; visual cylinder length=0.01 radius=0.006
- added link right_front_paw, mass 0.0005; collision cylinder length=0.01 radius=0.006; visual cylinder length=0.01 radius=0.006
- link left_lower_arm: mass 0.075 -> 0.017; geometry collision cylinder length=0.05 radius=0.003; visual cylinder length=0.05 radius=0.003
- link left_lower_leg: mass 0.075 -> 0.017; geometry collision cylinder length=0.05 radius=0.003; visual cylinder length=0.05 radius=0.003
- link left_upper_arm: mass 0.025 -> 0.005; geometry collision cylinder length=0.045 radius=0.003; visual cylinder length=0.045 radius=0.003
- link left_upper_leg: mass 0.025 -> 0.005; geometry collision cylinder length=0.045 radius=0.003; visual cylinder length=0.045 radius=0.003
- link right_lower_arm: mass 0.075 -> 0.017; geometry collision cylinder length=0.05 radius=0.003; visual cylinder length=0.05 radius=0.003
- link right_lower_leg: mass 0.075 -> 0.017; geometry collision cylinder length=0.05 radius=0.003; visual cylinder length=0.05 radius=0.003
- link right_upper_arm: mass 0.025 -> 0.005; geometry collision cylinder length=0.045 radius=0.003; visual cylinder length=0.045 radius=0.003
- link right_upper_leg: mass 0.025 -> 0.005; geometry collision cylinder length=0.045 radius=0.003; visual cylinder length=0.045 radius=0.003
- link torso: mass 0.2 -> 0.179; geometry collision box size=0.12 0.08 0.015; visual box size=0.12 0.08 0.015
Joints:
- added joint paw_back_left: type fixed, parent left_lower_leg, child left_back_paw, origin xyz=0.00 0.0 -0.05 rpy=0 -1.57 0
- added joint paw_back_right: type fixed, parent right_lower_leg, child right_back_paw, origin xyz=0.00 0.0 -0.05 rpy=0 -1.57 0
- added joint paw_front_left: type fixed, parent left_lower_arm, child left_front_paw, origin xyz=0.00 0.0 -0.05 rpy=0 -1.57 0
- added joint paw_front_right: type fixed, parent right_lower_arm, child right_front_paw, origin xyz=0.00 0.0 -0.05 rpy=0 -1.57 0
- joint elbow_left: origin xyz=0.00 0.00 -0.05 rpy=0 -1.57 0 -> xyz=0.00 -0.015 -0.045 rpy=0 -1.57 0
- joint elbow_right: origin xyz=0.00 0.00 -0.05 rpy=0 -1.57 0 -> xyz=0.00 0.015 -0.045 rpy=0 -1.57 0
- joint hip_left: limit lower=-1.57 upper=1.57 effort=0 velocity=0 -> lower=-1.57 upper=2.00 effort=0 velocity=0
- joint hip_right: limit lower=-1.57 upper=1.57 effort=0 velocity=0 -> lower=-1.57 upper=2.00 effort=0 velocity=0
- joint knee_left: origin xyz=0.00 0.00 -0.05 rpy=0 -1.57 0 -> xyz=0.00 -0.015 -0.045 rpy=0 -1.57 0
- joint knee_right: origin xyz=0.00 0.00 -0.05 rpy=0 -1.57 0 -> xyz=0.00 0.015 -0.045 rpy=0 -1.57 0
